Commit message: Fixing xacro values.

File: aliengo_description/xacro/robot.xacro (robot description, xacro)
@@ -114,8 +114,8 @@
     </link>
     <xacro:camera_sensor parent="base" camera_id="t265_link">
-        <origin xyz="-0.33118 0 0" rpy="0.244346 0.0 0"/>
+        <origin xyz="0.33118 0 0" rpy="0.244346 0.0 0"/>
     </xacro:camera_sensor>
     <xacro:camera_sensor parent="base" camera_id="d435_link">
-        <origin xyz="-0.061 0 0" rpy="0.244346 0.0 0"/>
+        <origin xyz="0.33118 0 -0.061" rpy="0.244346 0.0 0"/>
     </xacro:camera_sensor>
     <xacro:leg name="FR" mirror="-1" mirror_dae= "False" front_hind="1" front_hind_dae="True">

Commit message: Add pitch.

File: aliengo_description/xacro/robot.xacro (robot description, xacro)
@@ -114,8 +114,8 @@
     </link>
     <xacro:camera_sensor parent="base" camera_id="t265_link">
-        <origin xyz="0.33118 0 0" rpy="0.244346 0.0 0"/>
+        <origin xyz="0.33118 0 0" rpy="0 0.244346 0"/>
     </xacro:camera_sensor>
     <xacro:camera_sensor parent="base" camera_id="d435_link">
-        <origin xyz="0.33118 0 -0.061" rpy="0.244346 0.0 0"/>
+        <origin xyz="0.33118 0 -0.061" rpy="0 0.244346 0"/>
     </xacro:camera_sensor>
     <xacro:leg name="FR" mirror="-1" mirror_dae= "False" front_hind="1" front_hind_dae="True">

Commit message: Add possible fix

File: aliengo_description/xacro/robot.xacro (robot description, xacro)
@@ -113,5 +113,10 @@
         </collision>
     </link>
-    <xacro:camera_sensor parent="base" camera_id="t265_link">
+    <joint name="t265_joint" type="fixed">
+        <parent link="t265_pose_frame"/>
+        <child link="t265_link"/>
+        <origin rpy="0 0 0" xyz="0 0 0"/>
+    </joint>
+    <xacro:camera_sensor parent="base" camera_id="t265_pose_frame">
         <origin xyz="0.33118 0 0" rpy="0 0.244346 0"/>
     </xacro:camera_sensor>

Commit message: Fix.

File: aliengo_description/xacro/robot.xacro (robot description, xacro)
@@ -113,10 +113,5 @@
         </collision>
     </link>
-    <joint name="t265_joint" type="fixed">
-        <parent link="t265_pose_frame"/>
-        <child link="t265_link"/>
-        <origin rpy="0 0 0" xyz="0 0 0"/>
-    </joint>
-    <xacro:camera_sensor parent="base" camera_id="t265_pose_frame">
+    <xacro:camera_sensor parent="base" camera_id="t265_link">
         <origin xyz="0.33118 0 0" rpy="0 0.244346 0"/>
     </xacro:camera_sensor>

Commit message: Adapted robot xacro.

File: aliengo_description/xacro/robot.xacro (robot description, xacro)
@@ -113,9 +113,6 @@
         </collision>
     </link>
-    <xacro:camera_sensor parent="base" camera_id="t265_link">
-        <origin xyz="0.33118 0 0" rpy="0 0.244346 0"/>
-    </xacro:camera_sensor>
     <xacro:camera_sensor parent="base" camera_id="d435_link">
-        <origin xyz="0.33118 0 -0.061" rpy="0 0.244346 0"/>
+        <origin xyz="0.33118 0 -0.03462" rpy="0 0.244346 0"/>
     </xacro:camera_sensor>
     <xacro:leg name="FR" mirror="-1" mirror_dae= "False" front_hind="1" front_hind_dae="True">
